File: KiCad_files/2ND_PCB/10_LED_ARM1.kicad_sch (KiCad schematic)
At the start: 11 parts

Commit message: 07/09 upload, no ERC errors
Parts:
- added U1: ~, symbol spinning:LED_ARM
Changed lines of the file:
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@@
+	)
+	(symbol
+		(lib_id "spinning:LED_ARM")
+		(at 180.34 3.81 0)
+		(unit 1)
+		(exclude_from_sim no)
+		(in_bom yes)
+		(on_board yes)
+		(dnp no)
+		(fields_autoplaced yes)
+		(property "Reference" "U1"
+			(at 181.61 3.1749 0)
+			(effects
+				(font
+					(size 1.27 1.27)
+				)
+				(justify left)
+				(hide yes)
+			)
+		)
+		(property "Value" "~"
+			(at 181.61 5.08 0)
+			(effects
+				(font
+					(size 1.27 1.27)
+				)
+				(justify left)
+			)
+		)
+		(property "Footprint" ""
+			(at 180.34 3.81 0)
+			(effects
+				(font
+					(size 1.27 1.27)
+				)
+				(hide yes)
+			)
+		)
+		(property "Datasheet" ""
+			(at 180.34 3.81 0)
+			(effects
+				(font
+					(size 1.27 1.27)
+				)
+				(hide yes)
+			)
+		)
+		(property "Description" ""
+			(at 180.34 3.81 0)
+			(effects
+				(font
+					(size 1.27 1.27)
+				)
+				(hide yes)
+			)
+		)
+		(instances
+			(project ""
+				(path "/500a9f84-d59e-418d-bc4b-2142a90d742d/149f3120-9cd7-47ee-92dc-9bdec38b8376"
+					(reference "U1")
+					(unit 1)
+				)
+			)
+		)
 	)
 	(symbol
